File: Medidor_ruido_solar/Cargador_Balanceador/Cargador_Balanceador.sch (KiCad schematic (older format))
At the start: 8 parts, among them SW1 SW_SPDT, SW2 SW_SPDT, SW3 SW_SPDT

Commit message: Medidor_Ruido_Solar
Medidor_Ruido_Solar
Parts:
- added D3: 1N400X, symbol D_ALT
Connections:
- net at D1.1 (K), R1.2: no longer R2.1
- net at D1.2 (A), UX.3 (OUT): now also D3.2 (A)
- new net: D3.1 (K), R2.1
Other:
- moved on the sheet: D1
Changed lines of the file:
@@
 LIBS:contrib
 LIBS:valves
+LIBS:Cargador_Balanceador-cache
 EELAYER 25 0
 EELAYER END
@@
 L D_ALT D1
 U 1 1 5BDD9DC4
-P 3850 2700
-F 0 "D1" H 3850 2800 50  0000 C CNN
-F 1 "1N400X" H 3850 2600 50  0000 C CNN
-F 2 "" H 3850 2700 50  0001 C CNN
-F 3 "" H 3850 2700 50  0001 C CNN
-	1    3850 2700
-	-1   0    0    1
+P 4650 2650
+F 0 "D1" H 4650 2750 50  0000 C CNN
+F 1 "1N400X" H 4650 2550 50  0000 C CNN
+F 2 "" H 4650 2650 50  0001 C CNN
+F 3 "" H 4650 2650 50  0001 C CNN
+	1    4650 2650
+	0    -1   -1   0
 $EndComp
 $Comp
@@
 	1300 3450 3700 3450
 Wire Wire Line
-	2300 2700 3700 2700
-Wire Wire Line
-	4000 2700 4650 2700
-Wire Wire Line
 	4650 3250 5000 3250
 Wire Wire Line
@@
 $EndComp
 Wire Wire Line
-	4650 2700 4650 2850
-Wire Wire Line
-	4350 2850 4350 2700
-Connection ~ 4350 2700
+	4650 2800 4650 2850
 Wire Wire Line
 	4350 3150 4350 4350
@@
 Connection ~ 4650 4350
 Connection ~ 4650 3250
+$Comp
+L D_ALT D3
+U 1 1 5BDD9685
+P 4350 2650
+F 0 "D3" H 4350 2750 50  0000 C CNN
+F 1 "1N400X" H 4350 2550 50  0000 C CNN
+F 2 "" H 4350 2650 50  0001 C CNN
+F 3 "" H 4350 2650 50  0001 C CNN
+	1    4350 2650
+	0    -1   -1   0
+$EndComp
+Wire Wire Line
+	4350 2850 4350 2800
+Wire Wire Line
+	4650 2500 4650 2300
+Wire Wire Line
+	4650 2300 3850 2300
+Wire Wire Line
+	3850 2300 3850 2700
+Wire Wire Line
+	3850 2700 2300 2700
+Wire Wire Line
+	4350 2300 4350 2500
+Connection ~ 4350 2300
 $EndSCHEMATC
